File: project_digital_circuits.kicad_sch (KiCad schematic)
At the start: 53 parts, among them J1 Grove - universal connector 4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, J2 Conn_01x06_Pin, J3 Conn_01x06_Pin, P1 USB_C_Plug_USB2.0, P2 XT30PW-F, Q1 Si4214, Q2 Si4214, Q3 Si4214, SW1 SW_Push, U1 TB6612FNG, U2 LTC4365DDB, U3 LMR33630ADDA, U4 MPU-6050, U5 VL53L0CXV0DH1

Commit message: Correction of connection UART->USB and Status RGB led added
Parts:
- added C21, C22, C23: 100n, symbol Device:C
- added C24: 100u, symbol Device:C_Polarized
- added C25, C26: 47p, symbol Device:C
- added C27: 1u, symbol Device:C
- added D1: LED_RKGB, symbol Device:LED_RKGB
- added Q4, Q5, Q6: AO3400A, Package_TO_SOT_SMD:SOT-23, symbol Transistor_FET:AO3400A
- added R20, R21: 27, symbol Device:R
- added R22: 4k7, symbol Device:R
- added R23, R24: 10k, symbol Device:R
- added R25: 68, symbol Device:R
- added R26, R27: 15, symbol Device:R
- added R28, R29, R30: 220, symbol Device:R
- added U6: FT234XD-T, FT234XD-T:SON45P300X300X80-13N, symbol FT234XD-T:FT234XD-T
- C17, C20: value 0.1uF -> 0u1
- C18: value 10uF -> 10u
- gave numbers to parts that had none: 1
Connections:
- net +3.3V: now also C21.1, C22.1, C24.1, D1.2 (K), R24.1, U6.4 (VCC)
- net EN: now also C27.1, R24.2
- net GND: now also C20.1, C21.2, C22.2, C23.2, C24.2, C25.1, C26.2, C27.2, Q4.2 (S), Q5.2 (S), Q6.2 (S), R23.2, U6.13 (GND), U6.5 (GND); no longer C20.2
- net RX: now also U6.10 (RXD); no longer P1.A7 (D-)
- net TX: now also U6.7 (TXD); no longer P1.A6 (D+)
- net 2.5-13.5v: now reaches C19.1, U1.13 (VM2), U1.14 (VM3), U1.24 (VM1)
- net 2.5-13.5v: now also C20.2; no longer C20.1
- net GPIO_R: now reaches U7.19 (IO15)
- net GPIO_R: now also R30.2
- net GPIO_G: now reaches U7.20 (IO16)
- net GPIO_G: now also R29.2
- net GPIO_B: now reaches U7.21 (IO17)
- net GPIO_B: now also R28.2
- net VBUS: now reaches P1.A4 (VBUS), P1.A9 (VBUS), P1.B4 (VBUS), P1.B9 (VBUS)
- net VBUS: now also R22.2, R23.1
- new net: C25.2, P1.A6 (D+), R20.2
- new net: R22.1, U6.6 (CBUS0)
- new net: Q4.1 (G), R28.1
- new net: Q4.3 (D), R27.1
- new net: Q5.1 (G), R29.1
- new net: C26.1, P1.A7 (D-), R21.2
- new net: Q6.1 (G), R30.1
- new net: Q5.3 (D), R26.1
- new net: Q6.3 (D), R25.2
- new net 3v3OUT: U6.3 (3V3OUT)
- new net D+: R20.1, U6.12 (USBDP)
- new net D-: R21.1, U6.1 (USBDM)
- new net Drain_B: D1.4 (BA), R27.2
- new net Drain_G: D1.3 (GA), R26.2
- new net Drain_R: D1.1 (RA), R25.1
- new net VCCIO: C23.1, U6.2 (~{RESET}#), U6.9 (VCCIO)
- no-connect marks 4 -> 5
Other:
- note added: "Encoders connections"
- note added: "Motor A&B control"
- note added: "Stable power-up"
- note added: "Status RGB led"
- note removed: "Encoders"
- note removed: "Motors' control"
- moved on the sheet: C1, C10, C11, C12, C13, C14, C15, C16, C17, C18, C19, C2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

Commit message: Correction and final touches
Parts:
- added J4, J5, J6, J7: PADS_to_solder, symbol Connector:Conn_01x04_Socket
- added R1, R2: 4k7, symbol Device:R
- D1: value LED_RKGB -> KAA-3528RGBS-11
- J1: value Grove - universal connector 4-pin -> PADS_to_solder
Connections:
- net +5V is gone; now on net +3.3V: J1.2 (Pin_2)
- net VCC +3.3V is gone; now on net +3.3V: U5.1 (AVDDVCSEL), U5.11 (AVDD)
- net +3.3V: now also J4.2 (Pin_2), J5.2 (Pin_2), J6.2 (Pin_2), J7.2 (Pin_2), R1.1, R2.1
- net GND: now also J4.1 (Pin_1), J5.1 (Pin_1), J6.1 (Pin_1), J7.1 (Pin_1)
- net SCL: no longer J1.4 (Pin_4)
- net SDA: no longer J1.3 (Pin_3)
- net SCL_1: now reaches R12.2
- net SCL_1: now also U4.23 (SCL), U7.23 (IO19); no longer U4.24 (SDA)
- net SDA_1: now reaches R13.2
- net SDA_1: now also U4.24 (SDA), U7.22 (IO18); no longer U4.23 (SCL)
- net SDA_2: now reaches U7.24 (IO20)
- net SDA_2: now also J1.3 (Pin_3), J4.3 (Pin_3), J5.3 (Pin_3), J6.3 (Pin_3), J7.3 (Pin_3), R1.2
- net SCL_2: now reaches U7.25 (IO21)
- net SCL_2: now also J1.4 (Pin_4), J4.4 (Pin_4), J5.4 (Pin_4), J6.4 (Pin_4), J7.4 (Pin_4), R2.2
- no-connect marks 5 -> 27
Other:
- note added: "/ADDITONAL/Internals of distance measurement sensors"
- note added: "Connections to distance sensors"
- note added: "Micromouse"
- note removed: "Connection to distance sensor"
- note removed: "Usune jesli Pan powie ze nie potrzebne"
- moved on the sheet: C1, C10, C11, C12, C13, C14, C15, C16, C17, C18, C19, C2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

Commit message: Footprints added
Parts:
- removed D1: KAA-3528RGBS-11, symbol Device:LED_RKGB
- removed Q2, Q3: Si4214, Package_TO_SOT_THT:TO-92_Inline, symbol Transistor_FET:BS108
- removed R14, R15, R16, R17: 10k, symbol Device:R
- removed R18, R19: 47k, symbol Device:R
- removed U5: VL53L0CXV0DH1, Sensor_Distance:ST_VL53L1x, symbol Sensor_Distance:VL53L0CXV0DH1
- added D3: LED_RAGB, LED_SMD:KAA-3528RGBS-11, symbol Device:LED_RAGB
- C1, C10, C11, C12, C9: footprint (none) -> Capacitor_SMD:C_0805_2012Metric
- C13, C14, C15, C16, C17, C2, C20, C21, C22, C23, C27, C3, C5, C6, C7, C8: footprint (none) -> Capacitor_SMD:C_0603_1608Metric
- C18, C24, C4: footprint (none) -> Capacitor_SMD:C_1210_3225Metric
- C19: value 10uF -> 10u; footprint (none) -> Capacitor_SMD:C_1210_3225Metric
- C25, C26: footprint (none) -> Capacitor_SMD:C_0402_1005Metric
- J1, J4, J5, J6, J7: footprint (none) -> Connector:SMD_Pad 4x1
- J2, J3: footprint (none) -> Connector:SMD_Pad 6x1
- L1: footprint (none) -> Inductor_SMD:DR-125
- P1: footprint (none) -> Connector_USB:USB_C_Receptacle_GCT_USB4105-xx-A_16P_TopMnt_Horizontal
- P2: footprint XT30PW-F:AMASS_XT30PW-F -> Connector_AMASS:AMASS_XT30PW-F_1x02_P2.50mm_Horizontal
- R1, R11, R12, R13, R2, R24, R28, R29, R3, R30, R5, R9: footprint (none) -> Resistor_SMD:R_0402_1005Metric
- R20, R21, R7, R8: footprint (none) -> Resistor_SMD:R_0603_1608Metric
- R25: footprint (none) -> Resistor_SMD:R_1206_3216Metric
- R26, R27: footprint (none) -> Resistor_SMD:R_2010_5025Metric
- R4: value R0 -> 0; footprint (none) -> Resistor_SMD:R_2010_5025Metric
- R6: value 5M49 -> 5M6; footprint (none) -> Resistor_SMD:R_0603_1608Metric
- SW1: footprint (none) -> Button_Switch_SMD:SW_SPST_Omron_B3FS-100xP
- U6: footprint FT234XD-T:SON45P300X300X80-13N -> Package_DFN_QFN:SON45P300X300X80-13N
Connections:
- net 2.5-13.5v is gone; now on net 9.6-13v: C19.1, C20.2, U1.13 (VM2), U1.14 (VM3), U1.24 (VM1)
- net Drain_B is gone; now on net +3.3V: R27.2
- net Drain_G is gone; now on net +3.3V: R26.2
- net Drain_R is gone; now on net +3.3V: R25.1
- net GND: now also D3.2 (A); no longer Q4.2 (S), Q5.2 (S), Q6.2 (S)
- new net Source_B: D3.4 (BK), Q4.2 (S)
- new net Source_G: D3.3 (GK), Q5.2 (S)
- new net Source_R: D3.1 (RK), Q6.2 (S)
Other:
- note removed: "/ADDITONAL/Internals of distance measurement sensors"
- moved on the sheet: C7, Q4, Q5, Q6, R25, R26, R27, R28, R29, R30

Commit message: footprints changed
Parts:
- C1, C10, C11, C12, C9: footprint Capacitor_SMD:C_0805_2012Metric -> Capacitor_SMD:C_0603_1608Metric
- C24: footprint Capacitor_SMD:C_1210_3225Metric -> Capacitor_SMD:CP_Elec_5x5.4
- C4: footprint Capacitor_SMD:C_1210_3225Metric -> Capacitor_SMD:CP_Elec_6.3x5.8
Changed lines of the file:
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@@
 			)
 		)
-		(property "Footprint" "Capacitor_SMD:C_1210_3225Metric"
+		(property "Footprint" "Capacitor_SMD:CP_Elec_6.3x5.8"
 			(at 319.7352 106.68 0)
 			(effects
@@
 			)
 		)
-		(property "Footprint" "Capacitor_SMD:C_0805_2012Metric"
+		(property "Footprint" "Capacitor_SMD:C_0603_1608Metric"
 			(at 334.9752 171.45 0)
 			(effects
@@
 			)
 		)
-		(property "Footprint" "Capacitor_SMD:C_1210_3225Metric"
+		(property "Footprint" "Capacitor_SMD:CP_Elec_5x5.4"
 			(at 105.1052 204.47 0)
 			(effects
@@
 			)
 		)
-		(property "Footprint" "Capacitor_SMD:C_0805_2012Metric"
+		(property "Footprint" "Capacitor_SMD:C_0603_1608Metric"
 			(at 121.6152 96.52 0)
 			(effects
@@
 			)
 		)
-		(property "Footprint" "Capacitor_SMD:C_0805_2012Metric"
+		(property "Footprint" "Capacitor_SMD:C_0603_1608Metric"
 			(at 357.8352 171.45 0)
 			(effects
@@
 			)
 		)
-		(property "Footprint" "Capacitor_SMD:C_0805_2012Metric"
+		(property "Footprint" "Capacitor_SMD:C_0603_1608Metric"
 			(at 369.2652 171.45 0)
 			(effects
@@
 			)
 		)
-		(property "Footprint" "Capacitor_SMD:C_0805_2012Metric"
+		(property "Footprint" "Capacitor_SMD:C_0603_1608Metric"
 			(at 346.4052 171.45 0)
 			(effects

Commit message: footprints changed again
Parts:
- J2: footprint Connector:SMD_Pad 6x1 -> Connector:SMD_Pad 4x1
- R10, R22, R23: footprint (none) -> Resistor_SMD:R_0402_1005Metric
Changed lines of the file:
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@@
 			)
 		)
-		(property "Footprint" ""
+		(property "Footprint" "Resistor_SMD:R_0402_1005Metric"
 			(at 143.51 180.848 90)
 			(effects
@@
 			)
 		)
-		(property "Footprint" ""
+		(property "Footprint" "Resistor_SMD:R_0402_1005Metric"
 			(at 320.802 180.34 90)
 			(effects
@@
 			)
 		)
-		(property "Footprint" ""
+		(property "Footprint" "Resistor_SMD:R_0402_1005Metric"
 			(at 152.4 180.848 90)
 			(effects
@@
 			)
 		)
-		(property "Footprint" "Connector:SMD_Pad 6x1"
+		(property "Footprint" "Connector:SMD_Pad 4x1"
 			(at 125.73 31.75 0)
 			(effects
